File: kicad_project/airboard/airboard.kicad_sch (KiCad schematic)
At the start: 0 parts

Commit message: feat(kicad_project): add new libraries and update symbol and footprint tables
Parts:
- added C1: 0603_Fl0.35_R_885012106031, Capacitor_SMD_Wurth:C_Wurth_WCAP-CSGP-0603_Fl0.35_R, symbol Capacitor_Wurth_WCAP-CSGP:0603_Fl0.35_R_885012106031
- added D1: WE-TVS-SS_DFN1210-6L_824012823, WE-TVS-SS_DFN1210-6L_824012823:WE-TVS_DFN1210-6L, symbol WE-TVS-SS_DFN1210-6L_824012823:WE-TVS-SS_DFN1210-6L_824012823
- added J2: USB_C_Receptacle_USB2.0_14P, Eagle_WR-USB (rev25c):629722000214, symbol Connector:USB_C_Receptacle_USB2.0_14P
- added R1: 0402_560112110012, Resistor_SMD_Wurth:R_Wurth_WRIS-RSKS-0402, symbol Resistor_Wurth_WRIS-RSKS:0402_560112110012
- added R2, R3: 0603_R_560112116017, Resistor_SMD_Wurth:R_Wurth_WRIS-RSKS-0603_R, symbol Resistor_Wurth_WRIS-RSKS:0603_R_560112116017
- added R4, R5: 0603_R_560112116043, Resistor_SMD_Wurth:R_Wurth_WRIS-RSKS-0603_R, symbol Resistor_Wurth_WRIS-RSKS:0603_R_560112116043
- added U1: ESP32-C3-WROOM-02, RF_Module:ESP32-C3-WROOM-02, symbol RF_Module:ESP32-C3-WROOM-02
- added U2: DPS368, DPS368:LGA8S145X65P2X4_200X250X110-V, symbol DPS368:DPS368
Connections:
- new net: R4.2, U1.13 (IO18)
- new net: R5.2, U1.14 (IO19)
- new net: J2.B5 (CC2), R3.1
- new net: J2.A5 (CC1), R2.1
- new net +3.3V: C1.1, U1.1 (3V3)
- new net +5V: J2.A4 (VBUS), J2.A9 (VBUS), J2.B4 (VBUS), J2.B9 (VBUS)
- new net GND: C1.2, D1.3, J2.A1 (GND), J2.A12 (GND), J2.B1 (GND), J2.B12 (GND), J2.S1 (SHIELD), R2.2, R3.2, U1.19 (GND), U1.9 (GND)
- new net USB_DN: D1.1, J2.A7 (D-), J2.B7 (D-), R4.1
- new net USB_DP: D1.2, J2.A6 (D+), J2.B6 (D+), R5.1
